File: motor_driver/motor_driver.kicad_sch (KiCad schematic)
At the start: 20 parts, among them U1 A14-LC-TT, U2 DRV8833PWR, U3 LDL1117S50R_

Commit message: updated pcb schematic with changes from testing
Parts:
- added PGOOD1: LED, Resistor_SMD:R_1206_3216Metric, symbol Device:LED
- added R5: 1k, Resistor_SMD:R_1206_3216Metric, symbol Device:R
- U1: footprint A14_LC_TT:A14-LC-TT_ASM -> footprints:A14-LC-TT_ASM
- U2: footprint DRV8833PWR:PW16_TEX -> footprints:DRV8833PWR
- U3: footprint LDL1117S50R:SOT230P700X180-4N -> footprints:SOT230P700X180-4N
Connections:
- net 5V: now also R5.1
- net GND: now also PGOOD1.1 (K)
- new net: PGOOD1.2 (A), R5.2
